File: remote-powerOn.kicad_pcb (KiCad board)
At the start: 2 copper layers, 43 x 43 mm, 16 parts, among them K1 LMR2-3D, Q1 2N2222

Commit message: create changes.md update pcb
Parts:
- added refer2: LOGO, SilkScreen:smth, B.Cu at (138.5, 76.4)
- K1: footprint LMR2-3D:LMR2-3D -> Relay_THT:LMR2-3D
- Q1: value 2N2222 -> BC517
- moved PC1 9.05 mm to (136.7, 94.3)
- moved OUT1 9.04 mm to (127.7, 94.3)
- moved Q1 2.03 mm to (155.2, 75.0)
Connections:
- PC1 pad 1: /OUT1 -> /OUT2
- PC1 pad 2: /OUT2 -> /OUT1
- Q1 pad 1: /GND -> Net-(D3-A)
- Q1 pad 2: Net-(D3-A) -> Net-(Q1-B)
- Q1 pad 3: Net-(Q1-B) -> /GND
Routing:
- net /OUT2: track 23.3 -> 20.4 mm
- net /OUT1: track 17.3 -> 19.8 mm
- net Net-(D3-A): track 50.9 -> 49.5 mm
- net Net-(Q1-B): track 13.3 -> 12.0 mm
