File: remote-powerOn.kicad_sch (KiCad schematic)
At the start: 11 parts, among them K1 LMR2-3D, Q1 2N2222

Commit message: create changes.md update pcb
Parts:
- removed Q1: 2N2222, Package_TO_SOT_THT:TO-92_Inline, symbol Transistor_BJT:2SC1941
- added Q1: BC517, Package_TO_SOT_THT:TO-92_Inline, symbol Transistor_BJT:BC517
- K1: footprint LMR2-3D:LMR2-3D -> Relay_THT:LMR2-3D
Connections:
- net GND: now also Q1.3 (E)
- net OUT1: now also PC1.2 (Pin_2); no longer PC1.1 (Pin_1)
- net OUT2: now also PC1.1 (Pin_1); no longer PC1.2 (Pin_2)
- net at D3.2 (A), K1.16, OUT2.1 (K): now also Q1.1 (C)
- net at R3.2: now also Q1.2 (B)
Other:
- note removed: "BTN_PIN1"
- note removed: "BTN_PIN2"
- title: v1.1.0 Relay controller with GPIO  -> Relay controller with GPIO 
Changed lines of the file:
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@@
 	(paper "A4")
 	(title_block
-		(title "v1.1.0 Relay controller with GPIO ")
-		(date "2026-06-06")
-		(rev "JUN_2026")
-		(comment 4 "1.1.0: Fix pin headers footprint 1mm -> 2.54mm")
-	)
-	(text "BTN_PIN1"
-		(exclude_from_sim no)
-		(at 193.04 75.184 0)
-		(effects
-			(font
-				(size 1.27 1.27)
-			)
-		)
-	)
-	(text "BTN_PIN2"
-		(exclude_from_sim no)
-		(at 193.04 77.724 0)
-		(effects
-			(font
-				(size 1.27 1.27)
-			)
-		)
+		(title "Relay controller with GPIO ")
+		(date "2026-06-09")
+		(rev "1.2.1")
+		(comment 4 "For version changes check change.md")
 	)
 	(text_box "CIRCUIT\n"
@@
 	(wire
 		(pts
-			(xy 200.66 76.2) (xy 200.66 64.77)
-		)
-		(stroke
-			(width 0)
-			(type default)
-		)
-	)
-	(wire
-		(pts
 			(xy 144.78 99.06) (xy 149.86 99.06)
 		)
@@
 	(wire
 		(pts
+			(xy 198.12 76.2) (xy 198.12 67.31)
+		)
+		(stroke
+			(width 0)
+			(type default)
+		)
+	)
+	(wire
+		(pts
 			(xy 157.48 71.12) (xy 157.48 76.2)
 		)
@@
 	(wire
 		(pts
+			(xy 187.96 76.2) (xy 198.12 76.2)
+		)
+		(stroke
+			(width 0)
+			(type default)
+		)
+	)
+	(wire
+		(pts
 			(xy 121.92 66.04) (xy 121.92 69.85)
 		)
@@
 	(wire
 		(pts
+			(xy 91.44 113.03) (xy 107.95 113.03)
+		)
+		(stroke
+			(width 0)
+			(type default)
+		)
+	)
+	(wire
+		(pts
+			(xy 107.95 66.04) (xy 121.92 66.04)
+		)
+		(stroke
+			(width 0)
+			(type default)
+		)
+	)
+	(wire
+		(pts
+			(xy 107.95 77.47) (xy 107.95 83.82)
+		)
+		(stroke
+			(width 0)
+			(type default)
+		)
+	)
+	(wire
+		(pts
+			(xy 130.81 93.98) (xy 144.78 93.98)
+		)
+		(stroke
+			(width 0)
+			(type default)
+		)
+	)
+	(wire
+		(pts
+			(xy 144.78 91.44) (xy 144.78 93.98)
+		)
+		(stroke
+			(width 0)
+			(type default)
+		)
+	)
+	(wire
+		(pts
+			(xy 144.78 93.98) (xy 144.78 99.06)
+		)
+		(stroke
+			(width 0)
+			(type default)
+		)
+	)
+	(wire
+		(pts
+			(xy 91.44 66.04) (xy 107.95 66.04)
+		)
+		(stroke
+			(width 0)
+			(type default)
+		)
+	)
+	(wire
+		(pts
+			(xy 107.95 113.03) (xy 149.86 113.03)
+		)
+		(stroke
+			(width 0)
+			(type default)
+		)
+	)
+	(wire
+		(pts
+			(xy 187.96 88.9) (xy 196.85 88.9)
+		)
+		(stroke
+			(width 0)
+			(type default)
+		)
+	)
+	(wire
+		(pts
+			(xy 144.78 72.39) (xy 144.78 76.2)
+		)
+		(stroke
+			(width 0)
+			(type default)
+		)
+	)
+	(wire
+		(pts
+			(xy 121.92 66.04) (xy 144.78 66.04)
+		)
+		(stroke
+			(width 0)
+			(type default)
+		)
+	)
+	(wire
+		(pts
+			(xy 200.66 64.77) (xy 200.66 78.74)
+		)
+		(stroke
+			(width 0)
+			(type default)
+		)
+	)
+	(wire
+		(pts
+			(xy 154.94 91.44) (xy 154.94 95.25)
+		)
+		(stroke
+			(width 0)
+			(type default)
+		)
+	)
+	(wire
+		(pts
+			(xy 130.81 87.63) (xy 130.81 93.98)
+		)
+		(stroke
+			(width 0)
+			(type default)
+		)
+	)
+	(wire
+		(pts
+			(xy 187.96 86.36) (xy 196.85 86.36)
+		)
+		(stroke
+			(width 0)
+			(type default)
+		)
+	)
+	(wire
+		(pts
+			(xy 121.92 93.98) (xy 130.81 93.98)
+		)
+		(stroke
+			(width 0)
+			(type default)
+		)
+	)
+	(wire
+		(pts
 			(xy 187.96 64.77) (xy 200.66 64.77)
 		)
@@
 	(wire
 		(pts
-			(xy 91.44 113.03) (xy 107.95 113.03)
-		)
-		(stroke
-			(width 0)
-			(type default)
-		)
-	)
-	(wire
-		(pts
-			(xy 199.39 78.74) (xy 199.39 67.31)
-		)
-		(stroke
-			(width 0)
-			(type default)
-		)
-	)
-	(wire
-		(pts
-			(xy 107.95 66.04) (xy 121.92 66.04)
-		)
-		(stroke
-			(width 0)
-			(type default)
-		)
-	)
-	(wire
-		(pts
-			(xy 107.95 77.47) (xy 107.95 83.82)
-		)
-		(stroke
-			(width 0)
-			(type default)
-		)
-	)
-	(wire
-		(pts
-			(xy 130.81 93.98) (xy 144.78 93.98)
-		)
-		(stroke
-			(width 0)
-			(type default)
-		)
-	)
-	(wire
-		(pts
-			(xy 187.96 67.31) (xy 199.39 67.31)
-		)
-		(stroke
-			(width 0)
-			(type default)
-		)
-	)
-	(wire
-		(pts
-			(xy 144.78 91.44) (xy 144.78 93.98)
-		)
-		(stroke
-			(width 0)
-			(type default)
-		)
-	)
-	(wire
-		(pts
-			(xy 144.78 93.98) (xy 144.78 99.06)
-		)
-		(stroke
-			(width 0)
-			(type default)
-		)
-	)
-	(wire
-		(pts
-			(xy 91.44 66.04) (xy 107.95 66.04)
-		)
-		(stroke
-			(width 0)
-			(type default)
-		)
-	)
-	(wire
-		(pts
-			(xy 107.95 113.03) (xy 149.86 113.03)
-		)
-		(stroke
-			(width 0)
-			(type default)
-		)
-	)
-	(wire
-		(pts
-			(xy 187.96 88.9) (xy 196.85 88.9)
-		)
-		(stroke
-			(width 0)
-			(type default)
-		)
-	)
-	(wire
-		(pts
-			(xy 187.96 78.74) (xy 199.39 78.74)
-		)
-		(stroke
-			(width 0)
-			(type default)
-		)
-	)
-	(wire
-		(pts
-			(xy 144.78 72.39) (xy 144.78 76.2)
-		)
-		(stroke
-			(width 0)
-			(type default)
-		)
-	)
-	(wire
-		(pts
-			(xy 121.92 66.04) (xy 144.78 66.04)
-		)
-		(stroke
-			(width 0)
-			(type default)
-		)
-	)
-	(wire
-		(pts
-			(xy 154.94 91.44) (xy 154.94 95.25)
-		)
-		(stroke
-			(width 0)
-			(type default)
-		)
-	)
-	(wire
-		(pts
-			(xy 130.81 87.63) (xy 130.81 93.98)
-		)
-		(stroke
-			(width 0)
-			(type default)
-		)
-	)
-	(wire
-		(pts
-			(xy 187.96 86.36) (xy 196.85 86.36)
-		)
-		(stroke
-			(width 0)
-			(type default)
-		)
-	)
-	(wire
-		(pts
-			(xy 121.92 93.98) (xy 130.81 93.98)
-		)
-		(stroke
-			(width 0)
-			(type default)
-		)
-	)
-	(wire
-		(pts
 			(xy 121.92 77.47) (xy 121.92 83.82)
 		)
@@
 	(wire
 		(pts
+			(xy 187.96 67.31) (xy 198.12 67.31)
+		)
+		(stroke
+			(width 0)
+			(type default)
+		)
+	)
+	(wire
+		(pts
 			(xy 130.81 72.39) (xy 130.81 80.01)
 		)
@@
 	(wire
 		(pts
-			(xy 187.96 76.2) (xy 200.66 76.2)
+			(xy 200.66 78.74) (xy 187.96 78.74)
 		)
 		(stroke
@@
 			)
 		)
-		(property "Footprint" "LMR2-3D:LMR2-3D"
+		(property "Footprint" "Relay_THT:LMR2-3D"
 			(at 171.45 85.09 0)
 			(hide yes)
@@
 			)
 		)
-		(property "Datasheet" "http://omronfs.omron.com/en_US/ecb/products/pdf/en-g5v_2.pdf"
+		(property "Datasheet" "https://www.tme.eu/Document/cb95bab3047ea17130b1da862f2b7351/LMR-series.pdf"
 			(at 154.94 83.82 0)
 			(hide yes)
@@
 	)
 	(symbol
-		(lib_id "Transistor_BJT:2SC1941")
+		(lib_id "Transistor_BJT:BC517")
 		(at 147.32 104.14 0)
 		(unit 1)
@@
 			)
 		)
-		(property "Value" "2N2222"
+		(property "Value" "BC517"
 			(at 152.4 105.4099 0)
 			(show_name no)
@@
 			)
 		)
-		(property "Datasheet" "http://rtellason.com/transdata/2sc1941.pdf"
+		(property "Datasheet" "https://www.onsemi.com/pub/Collateral/BC517-D74Z-D.PDF"
 			(at 147.32 104.14 0)
 			(hide yes)
@@
 			)
 		)
-		(property "Description" "50mA Ic, 160V Vce, Audio High Voltage NPN Transistor, TO-92"
+		(property "Description" "1A Ic, 30V Vce, Darlington NPN Transistor, TO-92"
 			(at 147.32 104.14 0)
 			(hide yes)
-			(show_name no)
-			(do_not_autoplace no)
-			(effects
-				(font
-					(size 1.27 1.27)
-				)
-			)
-		)
-		(property "Sim.Device" "NPN"
-			(at 147.32 104.14 0)
-			(hide yes)
-			(show_name no)
-			(do_not_autoplace no)
-			(effects
-				(font
-					(size 1.27 1.27)
-				)
-			)
-		)
-		(property "Sim.Pins" "1=E 2=C 3=B"
-			(at 147.32 104.14 0)
-			(hide yes)
