File: kicad/remote-powerOn.kicad_sch (KiCad schematic)
At the start: 11 parts, among them K1 LMR2-3D, Q1 BC517

Commit message: v1.3.0
Parts:
- added H1, H2, H3, H4: MountingHole_Pad, MountingHole:MountingHole_2.7mm_M2.5_DIN965_Pad, symbol Mechanical:MountingHole_Pad
- added RV1: CA14NV12,5-10KA2020, Potentiometer_THT:Potentiometer_ACP_CA14V-15_Vertical_Hole, symbol Device:R_Potentiometer
- R1: value 1K -> 1k
Connections:
- net GND: now also H1.1, H2.1, H3.1, H4.1, RV1.3
- net at PWR1.2 (A): now also RV1.2; no longer R1.2
- new net: R1.2, RV1.1
Other:
- moved on the sheet: PWR1
